Commit message: controllers impact on simulated dynamics - updated models and ee wrench signal generation

File: assets/robots/fmrr_tecnobody/description/fmrr_tecnobody.urdf (robot description, URDF)
Before this commit: robot fmrr_tecnobody, 16 links, 15 joints
Links:
- link ee_link: mass 0.01 -> 5.0
- link flange_link: mass 0.01 -> 0.001
- link ft_link: mass 0.01 -> 0.001
- link link1: mass 0.2 -> 53.2093
- link link1_beam: mass 0.6 -> 0.001
- link link2: mass 0.2 -> 7.9491
- link link3: mass 0.97 -> 3.898

Commit message: controllers impact on simulated dynamics - ee wrench fixes for fmrr

File: assets/robots/fmrr_tecnobody/description/fmrr_tecnobody.urdf (robot description, URDF)
Before this commit: robot fmrr_tecnobody, 16 links, 15 joints
Joints:
- joint joint_x: limit lower=${-beam_lenght/2+2*radius} upper=${beam_lenght/2-2*radius} effort=1000 velocity=1 -> lower=${-beam_lenght/2+2*radius} upper=${beam_lenght/2-2*radius} effort=261.9 velocity=1
- joint joint_y: limit lower=${-beam_lenght/2+2*radius} upper=${beam_lenght/2-2*radius} effort=1000 velocity=1 -> lower=${-beam_lenght/2+2*radius} upper=${beam_lenght/2-2*radius} effort=261.9 velocity=1
- joint joint_z: limit lower=${-z_height/2} upper=${z_height/2} effort=1000 velocity=1 -> lower=${-z_height/2} upper=${z_height/2} effort=986.1 velocity=1
