Commit message: round 6 - first long run (iiwa and fmrr part 1)

File: assets/robots/kuka_lbr_iiwa_14_r820/description/kuka_lbr_iiwa_14_r820.urdf (robot description, URDF)
Before this commit: robot kuka_lbr_iiwa_14_r820, 9 links, 8 joints
Joints:
- joint iiwa_A1: limit lower=-2.9670597283903604 upper=2.9670597283903604 effort=200 velocity=1.4835298641951802 -> lower=-2.9670597283903604 upper=2.9670597283903604 effort=320 velocity=1.4835298641951802
- joint iiwa_A2: limit lower=-2.0943951023931953 upper=2.0943951023931953 effort=200 velocity=1.4835298641951802 -> lower=-2.0943951023931953 upper=2.0943951023931953 effort=320 velocity=1.4835298641951802
- joint iiwa_A3: limit lower=-2.9670597283903604 upper=2.9670597283903604 effort=200 velocity=1.7453292519943295 -> lower=-2.9670597283903604 upper=2.9670597283903604 effort=176 velocity=1.7453292519943295
- joint iiwa_A4: limit lower=-2.0943951023931953 upper=2.0943951023931953 effort=200 velocity=1.3089969389957472 -> lower=-2.0943951023931953 upper=2.0943951023931953 effort=176 velocity=1.3089969389957472
- joint iiwa_A5: limit lower=-2.9670597283903604 upper=2.9670597283903604 effort=200 velocity=2.2689280275926285 -> lower=-2.9670597283903604 upper=2.9670597283903604 effort=110 velocity=2.2689280275926285
- joint iiwa_A6: limit lower=-2.0943951023931953 upper=2.0943951023931953 effort=200 velocity=2.356194490192345 -> lower=-2.0943951023931953 upper=2.0943951023931953 effort=40 velocity=2.356194490192345
- joint iiwa_A7: limit lower=-3.0543261909900763 upper=3.0543261909900763 effort=200 velocity=2.356194490192345 -> lower=-3.0543261909900763 upper=3.0543261909900763 effort=40 velocity=2.356194490192345

File: assets/robots/kuka_lbr_iiwa_14_r820_table/description/kuka_lbr_iiwa_14_r820_table.urdf (robot description, URDF)
Before this commit: robot kuka_lbr_iiwa_14_r820_table, 10 links, 9 joints
Joints:
- joint iiwa_A1: limit lower=-2.9670597283903604 upper=2.9670597283903604 effort=200 velocity=1.4835298641951802 -> lower=-2.9670597283903604 upper=2.9670597283903604 effort=320 velocity=1.4835298641951802
- joint iiwa_A2: limit lower=-2.0943951023931953 upper=2.0943951023931953 effort=200 velocity=1.4835298641951802 -> lower=-2.0943951023931953 upper=2.0943951023931953 effort=320 velocity=1.4835298641951802
- joint iiwa_A3: limit lower=-2.9670597283903604 upper=2.9670597283903604 effort=200 velocity=1.7453292519943295 -> lower=-2.9670597283903604 upper=2.9670597283903604 effort=176 velocity=1.7453292519943295
- joint iiwa_A4: limit lower=-2.0943951023931953 upper=2.0943951023931953 effort=200 velocity=1.3089969389957472 -> lower=-2.0943951023931953 upper=2.0943951023931953 effort=176 velocity=1.3089969389957472
- joint iiwa_A5: limit lower=-2.9670597283903604 upper=2.9670597283903604 effort=200 velocity=2.2689280275926285 -> lower=-2.9670597283903604 upper=2.9670597283903604 effort=110 velocity=2.2689280275926285
- joint iiwa_A6: limit lower=-2.0943951023931953 upper=2.0943951023931953 effort=200 velocity=2.356194490192345 -> lower=-2.0943951023931953 upper=2.0943951023931953 effort=40 velocity=2.356194490192345
- joint iiwa_A7: limit lower=-3.0543261909900763 upper=3.0543261909900763 effort=200 velocity=2.356194490192345 -> lower=-3.0543261909900763 upper=3.0543261909900763 effort=40 velocity=2.356194490192345
